File: KiCad/SUMOBoard/SUMOBoard.kicad_pcb (KiCad board)
At the start: 2 copper layers, 89 x 26.9 mm, 8 parts, among them J5 Conn_01x20_Pin, M3 MountingHole, U1 Pico

Commit message: Build2作成
Parts:
- removed H2: MountingHole, MountingHole:MountingHole_3.2mm_M3
- removed J5: Conn_01x20_Pin, Connector_PinHeader_2.54mm:PinHeader_1x20_P2.54mm_Vertical
- removed mr8-C, mr8-D: Conn_01x03_Socket, Connector_JST:JST_XH_B3B-XH-A_1x03_P2.50mm_Vertical
- added D1: D, Diode_SMD:D_SMA_Handsoldering, B.Cu at (122.8, 123.5)
- added D2: LED, LED_SMD:LED_0603_1608Metric_Pad1.05x0.95mm_HandSolder, F.Cu at (194.9, 126.7)
- added D3: LED, LED_SMD:LED_0603_1608Metric_Pad1.05x0.95mm_HandSolder, F.Cu at (195.0, 134.3)
- added D4: D, Diode_SMD:D_SMA_Handsoldering, B.Cu at (138.8, 133.7)
- added J3: Conn_01x02, Connector_JST:JST_XH_B2B-XH-A_1x02_P2.50mm_Vertical, F.Cu at (129.9, 117.1)
- added J6: Conn_01x02, Connector_JST:JST_XH_B2B-XH-A_1x02_P2.50mm_Vertical, F.Cu at (202.4, 117.0)
- added J7: Conn_01x19_Pin, Connector_PinHeader_2.54mm:PinHeader_1x19_P2.54mm_Vertical, F.Cu at (147.5, 138.5)
- added R1: R, Resistor_SMD:R_0603_1608Metric_Pad0.98x0.95mm_HandSolder, F.Cu at (197.2, 124.8)
- added R2: R, Resistor_SMD:R_0603_1608Metric_Pad0.98x0.95mm_HandSolder, F.Cu at (197.2, 132.4)
- added U1: ~, 0AS1R5-4805:0AS1R5-4805, F.Cu at (119.0, 127.6)
- J1: renamed from mr8-B; value Conn_01x03_Socket -> Conn_01x03
- J4: renamed from mr8-A; value Conn_01x03_Socket -> Conn_01x03
- moved J1 7.72 mm to (130.0, 124.8), turned to 0 degrees
- moved J4 5.78 mm to (130.0, 133.7), turned to 0 degrees
- renumbered M3 to H1, U1 to U2
Connections:
- J1 pad 1: mr8-B -> GND
- J1 pad 2: +3.3V -> +5V
- J1 pad 3: GND -> mr8-C
- J4 pad 1: mr8-A -> GND
- J4 pad 2: +3.3V -> +5V
- J4 pad 3: GND -> mr8-A
- U2 pad 1: Pico-TX -> Odrive-RX
- U2 pad 10: unconnected-(U1-GPIO7-Pad10)_0 -> LED2
- U2 pad 2: Pico-RX -> Odrive-TX
- U2 pad 36: unconnected-(U1-3V3-Pad36)_0 -> +3.3V
- U2 pad 39: +3.3V -> +5V
- U2 pad 5: mr8-B -> mr8-C
- U2 pad 6: mr8-C -> mr8-G
- U2 pad 7: mr8-D -> mr8-H
- U2 pad 9: unconnected-(U1-GPIO6-Pad9) -> LED1
Routing:
- net +3.3V: track 172.7 -> 0.00 mm
- net +5V: track 0.00 -> 107.8 mm, vias 0 -> 3
- net mr8-D: track 60.5 -> 0.00 mm
- net mr8-B: track 59.8 -> 0.00 mm
- net LED2: track 0.00 -> 38.6 mm, vias 0 -> 2
- net Odrive-RX: track 0.00 -> 38.5 mm, vias 0 -> 1
- net Odrive-TX: track 0.00 -> 34.6 mm, vias 0 -> 2
- net LED1: track 0.00 -> 32.3 mm, vias 0 -> 2
- net +BATT: track 0.00 -> 18.8 mm
- net mr8-C: track 63.9 -> 48.9 mm
- net Net-(D3-A): track 0.00 -> 2.23 mm
- net Net-(D2-A): track 0.00 -> 2.11 mm
- net mr8-A: track 55.7 -> 57.6 mm
- net GND: vias 0 -> 66
- net (no net): vias 1 -> 0
Other:
- board size 89 x 26.9 mm -> 96.5 x 26.9 mm
- board text added: "+BATT"
- board text added: "Back Converter"
- board text added: "Build 2"
- board text added: "Capacitor"
- board text added: "Raspberry Pi Pico"
- board text added: "STATUS"
- board text added: "TASK"
- board text added: "ch A"
- board text added: "ch C"
- board text removed: "Build 1"
